File: Circuit/ARM_Debug_AdapterB.kicad_pcb (KiCad board)
At the start: 2 copper layers, 82.5 x 49.5 mm, 12 parts, among them J1 HDR-2.54 Male 2x10, J2 HDR-2.54 Male 2x7, J3 HDR-1.27 Male 2x7, J4 HDR-1.27 Male 2x5, J5 HDR-1.27 Male 2x5, J6 HDR-2.54 Male 2x6, J7 HDR-2.54 Male 1x6

Commit message: update PCB Trace Routing
Parts:
- JP2, JP3: moved to B.Cu
- moved JP3 8.25 mm to (173.3, 111.1)
- moved JP1 0.91 mm to (154.2, 83.7), turned to 0 degrees
Routing:
- net /NRST/NMCLR: track 0.00 -> 101.4 mm, vias 0 -> 4
- net /TMS/PGC/SWCLK: track 0.00 -> 98.1 mm, vias 0 -> 2
- net /TDO/PGD/SWO: track 11.8 -> 107.9 mm, vias 0 -> 6
- net /TMS/SWDIO: track 22.7 -> 118.6 mm, vias 0 -> 2
- net /TDI: track 0.00 -> 95.7 mm, vias 0 -> 3
- net /VDD/VTref: track 8.78 -> 95.5 mm, vias 0 -> 3
- net /JCLK: track 0.00 -> 39.8 mm, vias 0 -> 1
- net /VCP_RX: track 0.00 -> 26.0 mm, vias 0 -> 1
- net /VCP_TX: track 0.00 -> 22.9 mm
- net Net-(J3-Pin_11): track 0.00 -> 4.96 mm
- net Net-(J7-Pin_3): track 0.00 -> 4.46 mm

Commit message: Completed PCB routing
Parts:
- moved JP3 1.13 mm to (172.2, 111.1), turned to 180 degrees
Routing:
- net /TDO/PGD/SWO: track 107.9 -> 140.2 mm
- net /VDD/VTref: track 95.5 -> 124.6 mm, vias 3 -> 4
- net Net-(J7-Pin_3): track 4.46 -> 8.72 mm
- net /TMS/PGC/SWCLK: track 98.1 -> 98.8 mm
- net GNDREF: vias 0 -> 55
- added copper zone on B.Cu, net GNDREF
- added copper zone on F.Cu, net GNDREF
